Commit message: Fixed roll/strafe and depth/pitch thruster directions in structures.urdf for dummy_robot. Fixes #5

File: auv_model/dummy_robot/structures.urdf (robot description, URDF)
Before this commit: robot dummy_robot, 13 links, 12 joints
Joints:
- joint hull_to_thruster1: origin xyz=-0.3  0.0 0 rpy=0 1.57079 0 -> xyz=-0.3  0.0 0 rpy=0 -1.57079 0
- joint hull_to_thruster2: origin xyz=0.3  0.0 0 rpy=0 1.57079 0 -> xyz=0.3  0.0 0 rpy=0 -1.57079 0
- joint hull_to_thruster3: origin xyz=0 0 0.15 rpy=0 0 -1.57079 -> xyz=0 0 0.15 rpy=0 0 1.57079
- joint hull_to_thruster4: origin xyz=0 0 -0.15 rpy=0 0 1.57079 -> xyz=0 0 -0.15 rpy=0 0 -1.57079

Commit message: Added center of mass and center of volume to structures.urdf for dummy_robot.

File: auv_model/dummy_robot/structures.urdf (robot description, URDF)
Before this commit: robot dummy_robot, 13 links, 12 joints
Links:
- added link cm_link
- added link cv_link
Joints:
- added joint cm_to_cv: type fixed, parent cm_link, child cv_link, origin xyz=0.0  0.0 0.1 rpy=0 0 0
- added joint cm_to_hull: type fixed, parent cm_link, child hull_link, origin xyz=0.0  0.0 0.0 rpy=0 0 0

Commit message: Fixed missing value in dummy_thruster map, added stl model to dummy_robot and modified urdf to incorporate it.

File: auv_model/dummy_robot/structures.urdf (robot description, URDF)
Before this commit: robot dummy_robot, 15 links, 14 joints
Links:
- link hull_link: geometry visual mesh filename=package://auv_model/dummy_robot/stl/seabee3.STL
Joints:
- joint cm_to_hull: origin xyz=0.0  0.0 0.0 rpy=0 0 0 -> xyz=0.0 0.0 0.0 rpy=0 0 0
