Commit message: Fixed stl model path in seabee3 structures.urdf, fixed sign for gravity constant.

File: auv_model/seabee3/structures.urdf (robot description, URDF)
Before this commit: robot seabee3, 9 links, 8 joints
Links:
- link hull_link: geometry visual mesh filename=package://auv_model/seabee3/stl/seabee3.STL

Commit message: Added camera transforms to structures.urdf and changed naming convention. Added stl object_model package with stl files for some competition objects.

File: auv_model/seabee3/structures.urdf (robot description, URDF)
Before this commit: robot seabee3, 9 links, 8 joints
Links:
- removed link cm_link
- removed link cv_link
- removed link hull_link
- removed link thruster1_link
- removed link thruster2_link
- removed link thruster3_link
- removed link thruster4_link
- removed link thruster5_link
- removed link thruster6_link
- added link robot/cameras/downward/left
- added link robot/cameras/downward/right
- added link robot/cameras/forward/left
- added link robot/cameras/forward/right
- added link robot/structures/cm
- added link robot/structures/cv
- added link robot/structures/hull; visual mesh filename=package://auv_model/seabee3/stl/seabee3.STL
- added link robot/thrusters/thruster1
- added link robot/thrusters/thruster2
- added link robot/thrusters/thruster3
- added link robot/thrusters/thruster4
- added link robot/thrusters/thruster5
- added link robot/thrusters/thruster6
Joints:
- added joint hull_to_camera_downward_left: type fixed, parent robot/structures/hull, child robot/cameras/downward/left, origin xyz=0.0 0.189596 -0.094078 rpy=3.141592 0 0
- added joint hull_to_camera_downward_right: type fixed, parent robot/structures/hull, child robot/cameras/downward/right, origin xyz=0.0 -0.189596 -0.094078 rpy=3.141592 0 0
- added joint hull_to_camera_forward_left: type fixed, parent robot/structures/hull, child robot/cameras/forward/left, origin xyz=0.273819 0.189038 0.0 rpy=0 -1.57079 3.141592
- added joint hull_to_camera_forward_right: type fixed, parent robot/structures/hull, child robot/cameras/forward/right, origin xyz=0.273819 -0.189038 0.0 rpy=0 -1.57079 3.141592
- joint cm_to_hull: child hull_link -> robot/structures/hull; parent cm_link -> robot/structures/cm
- joint hull_to_cv: child cv_link -> robot/structures/cv; parent hull_link -> robot/structures/hull
- joint hull_to_thruster1: child thruster1_link -> robot/thrusters/thruster1; parent hull_link -> robot/structures/hull
- joint hull_to_thruster2: child thruster2_link -> robot/thrusters/thruster2; parent hull_link -> robot/structures/hull
- joint hull_to_thruster3: child thruster3_link -> robot/thrusters/thruster3; parent hull_link -> robot/structures/hull
- joint hull_to_thruster4: child thruster4_link -> robot/thrusters/thruster4; parent hull_link -> robot/structures/hull
- joint hull_to_thruster5: child thruster5_link -> robot/thrusters/thruster5; parent hull_link -> robot/structures/hull
- joint hull_to_thruster6: child thruster6_link -> robot/thrusters/thruster6; parent hull_link -> robot/structures/hull

Commit message: Changed camera rotation to reflect image frame.

File: auv_model/seabee3/structures.urdf (robot description, URDF)
Before this commit: robot seabee3, 13 links, 12 joints
Joints:
- joint hull_to_camera_downward_left: origin xyz=0.0 0.189596 -0.094078 rpy=3.141592 0 0 -> xyz=0.0 0.189596 -0.094078 rpy=0 3.141592 1.57079
- joint hull_to_camera_downward_right: origin xyz=0.0 -0.189596 -0.094078 rpy=3.141592 0 0 -> xyz=0.0 -0.189596 -0.094078 rpy=0 3.141592 1.57079
- joint hull_to_camera_forward_left: origin xyz=0.273819 0.189038 0.0 rpy=0 -1.57079 3.141592 -> xyz=0.273819 0.189038 0.0 rpy=-1.57079 0 -1.57079
- joint hull_to_camera_forward_right: origin xyz=0.273819 -0.189038 0.0 rpy=0 -1.57079 3.141592 -> xyz=0.273819 -0.189038 0.0 rpy=-1.57079 0 -1.57079

Commit message: Pulled over seabee structures updates from unstable, newer camera1/2 models, removed old teleop_config package.

File: auv_model/seabee3/structures.urdf (robot description, URDF)
Before this commit: robot seabee3, 9 links, 8 joints
Links:
- removed link cm_link
- removed link cv_link
- removed link hull_link
- removed link thruster1_link
- removed link thruster2_link
- removed link thruster3_link
- removed link thruster4_link
- removed link thruster5_link
- removed link thruster6_link
- added link robot/cameras/downward/left
- added link robot/cameras/downward/right
- added link robot/cameras/forward/left
- added link robot/cameras/forward/right
- added link robot/structures/cm
- added link robot/structures/cv
- added link robot/structures/hull; visual mesh filename=package://auv_model/seabee3/stl/seabee3.STL
- added link robot/thrusters/thruster1
- added link robot/thrusters/thruster2
- added link robot/thrusters/thruster3
- added link robot/thrusters/thruster4
- added link robot/thrusters/thruster5
- added link robot/thrusters/thruster6
Joints:
- added joint hull_to_camera_downward_left: type fixed, parent robot/structures/hull, child robot/cameras/downward/left, origin xyz=0.0 0.189596 -0.094078 rpy=0 3.141592 1.57079
- added joint hull_to_camera_downward_right: type fixed, parent robot/structures/hull, child robot/cameras/downward/right, origin xyz=0.0 -0.189596 -0.094078 rpy=0 3.141592 1.57079
- added joint hull_to_camera_forward_left: type fixed, parent robot/structures/hull, child robot/cameras/forward/left, origin xyz=0.273819 0.189038 0.0 rpy=-1.57079 0 -1.57079
- added joint hull_to_camera_forward_right: type fixed, parent robot/structures/hull, child robot/cameras/forward/right, origin xyz=0.273819 -0.189038 0.0 rpy=-1.57079 0 -1.57079
- joint cm_to_hull: child hull_link -> robot/structures/hull; parent cm_link -> robot/structures/cm
- joint hull_to_cv: child cv_link -> robot/structures/cv; parent hull_link -> robot/structures/hull
- joint hull_to_thruster1: child thruster1_link -> robot/thrusters/thruster1; parent hull_link -> robot/structures/hull
- joint hull_to_thruster2: child thruster2_link -> robot/thrusters/thruster2; parent hull_link -> robot/structures/hull
- joint hull_to_thruster3: child thruster3_link -> robot/thrusters/thruster3; parent hull_link -> robot/structures/hull
- joint hull_to_thruster4: child thruster4_link -> robot/thrusters/thruster4; parent hull_link -> robot/structures/hull
- joint hull_to_thruster5: child thruster5_link -> robot/thrusters/thruster5; parent hull_link -> robot/structures/hull
- joint hull_to_thruster6: child thruster6_link -> robot/thrusters/thruster6; parent hull_link -> robot/structures/hull

Commit message: Added better Pi values to structures definitions.

File: auv_model/seabee3/structures.urdf (robot description, URDF)
Before this commit: robot seabee3, 13 links, 12 joints
Joints:
- joint hull_to_camera_downward_left: origin xyz=0.0 0.189596 -0.094078 rpy=0 3.141592 1.57079 -> xyz=0.0 0.189596 -0.094078 rpy=0 3.1415926535897932384626433832795028841971693993751 1.5707963267948965579989817342720925807952880859375
- joint hull_to_camera_downward_right: origin xyz=0.0 -0.189596 -0.094078 rpy=0 3.141592 1.57079 -> xyz=0.0 -0.189596 -0.094078 rpy=0 3.1415926535897932384626433832795028841971693993751 1.5707963267948965579989817342720925807952880859375
- joint hull_to_camera_forward_left: origin xyz=0.273819 0.189038 0.0 rpy=-1.57079 0 -1.57079 -> xyz=0.273819 0.189038 0.0 rpy=-1.5707963267948965579989817342720925807952880859375 0 -1.5707963267948965579989817342720925807952880859375
- joint hull_to_camera_forward_right: origin xyz=0.273819 -0.189038 0.0 rpy=-1.57079 0 -1.57079 -> xyz=0.273819 -0.189038 0.0 rpy=-1.5707963267948965579989817342720925807952880859375 0 -1.5707963267948965579989817342720925807952880859375
- joint hull_to_thruster1: origin xyz=-0.32740  0.000421 -0.049628 rpy=0 -1.57079 0 -> xyz=-0.32740  0.000421 -0.049628 rpy=0 -1.5707963267948965579989817342720925807952880859375 0
- joint hull_to_thruster2: origin xyz=0.32740  -0.000421 -0.049618 rpy=0 -1.57079 0 -> xyz=0.32740  -0.000421 -0.049618 rpy=0 -1.5707963267948965579989817342720925807952880859375 0
- joint hull_to_thruster3: origin xyz=0.001304 -0.0499614 0.202502 rpy=0 0 1.57079 -> xyz=0.001304 -0.0499614 0.202502 rpy=0 0 1.5707963267948965579989817342720925807952880859375
- joint hull_to_thruster4: origin xyz=0.001304 0.050038 -0.202273 rpy=0 0 -1.57079 -> xyz=0.001304 0.050038 -0.202273 rpy=0 0 -1.5707963267948965579989817342720925807952880859375
